File: PCB/DoMo-pcb.sch (KiCad schematic (older format))
At the start: 8 parts, among them SW1 SW_Push, U1 ATmega32U4-AU, Y1 16MHz

Commit message: create decoupling capacitors
Parts:
- added C3: 1uF, symbol Device:C_Small
- added C4, C5, C6: 0.1uF, symbol Device:C_Small
- added C7: 10uF, symbol Device:C_Small
- added R4: 22ohm, symbol Device:R_Small
- R3: value 10k -> 22ohm
Connections:
- wire segments 33 -> 56
Other:
- note added: "Decoupling Capacitors"
Changed lines of the file:
@@
 	0    1    1    0
-$EndComp
-$Comp
-L Device:R_Small R3
-U 1 1 5F04C82D
-P 1950 2500
-F 0 "R3" V 2146 2500 50  0000 C CNN
-F 1 "10k" V 2055 2500 50  0000 C CNN
-F 2 "" H 1950 2500 50  0001 C CNN
-F 3 "~" H 1950 2500 50  0001 C CNN
-	1    1950 2500
-	0    -1   -1   0
 $EndComp
 Wire Wire Line
 	2250 1000 2250 1150
-$Comp
-L power:+5V #PWR?
-U 1 1 5F04BA07
-P 2250 1000
-F 0 "#PWR?" H 2250 850 50  0001 C CNN
-F 1 "+5V" H 2265 1173 50  0000 C CNN
-F 2 "" H 2250 1000 50  0001 C CNN
-F 3 "" H 2250 1000 50  0001 C CNN
-	1    2250 1000
-	1    0    0    -1
-$EndComp
 $Comp
 L Device:R_Small R2
@@
 	1    0    0    -1
 $EndComp
-Text Notes 700  650  0    50   ~ 0
+Text Notes 950  750  0    50   ~ 0
 MCU
+$Comp
+L power:+5V #PWR?
+U 1 1 5F04BA07
+P 2250 1000
+F 0 "#PWR?" H 2250 850 50  0001 C CNN
+F 1 "+5V" H 2265 1173 50  0000 C CNN
+F 2 "" H 2250 1000 50  0001 C CNN
+F 3 "" H 2250 1000 50  0001 C CNN
+	1    2250 1000
+	1    0    0    -1
+$EndComp
+$Comp
+L Device:C_Small C3
+U 1 1 5EFFD535
+P 2150 2950
+F 0 "C3" H 2242 2996 50  0000 L CNN
+F 1 "1uF" H 2242 2905 50  0000 L CNN
+F 2 "" H 2150 2950 50  0001 C CNN
+F 3 "~" H 2150 2950 50  0001 C CNN
+	1    2150 2950
+	1    0    0    -1
+$EndComp
+$Comp
+L power:GND #PWR?
+U 1 1 5EFFEC28
+P 2150 3150
+F 0 "#PWR?" H 2150 2900 50  0001 C CNN
+F 1 "GND" H 2155 2977 50  0000 C CNN
+F 2 "" H 2150 3150 50  0001 C CNN
+F 3 "" H 2150 3150 50  0001 C CNN
+	1    2150 3150
+	1    0    0    -1
+$EndComp
+Wire Wire Line
+	2450 2800 2150 2800
+Wire Wire Line
+	2150 2800 2150 2850
+Wire Wire Line
+	2150 3050 2150 3150
+$Comp
+L Device:R_Small R3
+U 1 1 5F001B6F
+P 1850 2600
+F 0 "R3" V 1950 2600 50  0000 C CNN
+F 1 "22ohm" V 2050 2600 50  0000 C CNN
+F 2 "" H 1850 2600 50  0001 C CNN
+F 3 "~" H 1850 2600 50  0001 C CNN
+	1    1850 2600
+	0    1    1    0
+$EndComp
+$Comp
+L Device:R_Small R4
+U 1 1 5F004BAC
+P 1850 2500
+F 0 "R4" V 1654 2500 50  0000 C CNN
+F 1 "22ohm" V 1745 2500 50  0000 C CNN
+F 2 "" H 1850 2500 50  0001 C CNN
+F 3 "~" H 1850 2500 50  0001 C CNN
+	1    1850 2500
+	0    1    1    0
+$EndComp
+Wire Wire Line
+	2450 2600 1950 2600
+Wire Wire Line
+	2450 2500 1950 2500
+$Comp
+L Device:C_Small C4
+U 1 1 5F006977
+P 1450 6600
+F 0 "C4" H 1542 6646 50  0000 L CNN
+F 1 "0.1uF" H 1542 6555 50  0000 L CNN
+F 2 "" H 1450 6600 50  0001 C CNN
+F 3 "~" H 1450 6600 50  0001 C CNN
+	1    1450 6600
+	1    0    0    -1
+$EndComp
+$Comp
+L Device:C_Small C5
+U 1 1 5F00730F
+P 1900 6600
+F 0 "C5" H 1992 6646 50  0000 L CNN
+F 1 "0.1uF" H 1992 6555 50  0000 L CNN
+F 2 "" H 1900 6600 50  0001 C CNN
+F 3 "~" H 1900 6600 50  0001 C CNN
+	1    1900 6600
+	1    0    0    -1
+$EndComp
+$Comp
+L Device:C_Small C6
+U 1 1 5F0078BE
+P 2350 6600
+F 0 "C6" H 2442 6646 50  0000 L CNN
+F 1 "0.1uF" H 2442 6555 50  0000 L CNN
+F 2 "" H 2350 6600 50  0001 C CNN
+F 3 "~" H 2350 6600 50  0001 C CNN
+	1    2350 6600
+	1    0    0    -1
+$EndComp
+$Comp
+L Device:C_Small C7
+U 1 1 5F007D2B
+P 2800 6600
+F 0 "C7" H 2708 6554 50  0000 R CNN
+F 1 "10uF" H 2708 6645 50  0000 R CNN
+F 2 "" H 2800 6600 50  0001 C CNN
+F 3 "~" H 2800 6600 50  0001 C CNN
+	1    2800 6600
+	-1   0    0    1
+$EndComp
+$Comp
+L power:+5V #PWR?
+U 1 1 5F008F2B
+P 2150 6300
+F 0 "#PWR?" H 2150 6150 50  0001 C CNN
+F 1 "+5V" H 2165 6473 50  0000 C CNN
+F 2 "" H 2150 6300 50  0001 C CNN
+F 3 "" H 2150 6300 50  0001 C CNN
+	1    2150 6300
+	1    0    0    -1
+$EndComp
+$Comp
+L power:GND #PWR?
+U 1 1 5F00B1AD
+P 2150 6950
+F 0 "#PWR?" H 2150 6700 50  0001 C CNN
+F 1 "GND" H 2155 6777 50  0000 C CNN
+F 2 "" H 2150 6950 50  0001 C CNN
+F 3 "" H 2150 6950 50  0001 C CNN
+	1    2150 6950
+	1    0    0    -1
+$EndComp
+Wire Wire Line
+	1450 6500 1450 6400
+Wire Wire Line
+	1450 6400 1900 6400
+Wire Wire Line
+	2150 6400 2150 6300
+Wire Wire Line
+	1900 6500 1900 6400
+Connection ~ 1900 6400
+Wire Wire Line
+	1900 6400 2150 6400
+Wire Wire Line
+	2150 6400 2350 6400
+Wire Wire Line
+	2800 6400 2800 6500
+Connection ~ 2150 6400
+Wire Wire Line
+	2350 6500 2350 6400
+Connection ~ 2350 6400
+Wire Wire Line
+	2350 6400 2800 6400
+Wire Wire Line
+	2800 6700 2800 6800
+Wire Wire Line
+	2800 6800 2350 6800
+Wire Wire Line
+	1450 6800 1450 6700
+Wire Wire Line
+	1900 6700 1900 6800
+Connection ~ 1900 6800
+Wire Wire Line
+	1900 6800 1450 6800
+Wire Wire Line
+	2350 6700 2350 6800
+Connection ~ 2350 6800
+Wire Wire Line
+	2350 6800 2150 6800
+Wire Wire Line
+	2150 6800 2150 6950
+Connection ~ 2150 6800
+Wire Wire Line
+	2150 6800 1900 6800
+Text Notes 1050 5950 0    50   ~ 0
+Decoupling Capacitors
+Wire Notes Line
+	500  5350 4750 5350
+Wire Notes Line
+	4750 5350 4750 500
+Wire Notes Line
+	3650 5350 3650 7700
 $EndSCHEMATC

Commit message: create rotary encoder
Parts:
- added SW2: Rotary_Encoder, symbol Device:Rotary_Encoder
Connections:
- net labels added: D+, D-, EN1, EN2
- wire segments 56 -> 62
Other:
- note added: "Rotary Encoder"
- moved on the sheet: SW1

Commit message: create OLED pins
Parts:
- added JOLED1: Conn_01x04, symbol Connector_Generic:Conn_01x04
Connections:
- net labels added: SCL, SDA
- wire segments 62 -> 68
Other:
- note added: "OLED"
- moved on the sheet: SW1

Commit message: change mcu to pro micro
Parts:
- removed C1, C2: 22p, symbol Device:C_Small
- removed C3: 1uF, symbol Device:C_Small
- removed C4, C5, C6: 0.1uF, symbol Device:C_Small
- removed C7: 10uF, symbol Device:C_Small
- removed R1, R2: 10k, symbol Device:R_Small
- removed R3, R4: 22ohm, symbol Device:R_Small
- removed SW1: SW_Push, symbol Switch:SW_Push
- removed SW2: Rotary_Encoder, symbol Device:Rotary_Encoder
- removed U1: ATmega32U4-AU, Package_QFP:TQFP-44_10x10mm_P0.8mm, symbol MCU_Microchip_ATmega:ATmega32U4-AU
- removed Y1: 16MHz, symbol Device:Crystal_GND24_Small
- added SW0: SW_Push, symbol Switch:SW_Push
- added SW1: Rotary_Encoder_Switch, symbol Device:Rotary_Encoder_Switch
- added U0: ProMicro, symbol keebio:ProMicro
- renumbered JOLED1 to JOLED0
Connections:
- net labels added: C0, C1, C2, EN0, LEDS, R0, R1, R2, RST, VCC
- net labels removed: +5V, D+, D-, EN2
- wire segments 68 -> 30
Other:
- note added: "RESET"
- note added: "ROTARY ENCODER"
- note removed: "Decoupling Capacitors"
- note removed: "Rotary Encoder"
- moved on the sheet: JOLED0

Commit message: create LEDS
Parts:
- added LED0, LED1, LED2, LED3, LED4: WS2812B, LED_SMD:LED_WS2812B_PLCC4_5.0x5.0mm_P3.2mm, symbol LED:WS2812B
Connections:
- net GND: now also LED0.3 (VSS), LED1.3 (VSS), LED2.3 (VSS), LED3.3 (VSS), LED4.3 (VSS)
- net LEDS: now also U0.1 (TX0/PD3), LED0.4 (DIN); no longer U0.20 (A3/PF4)
- net VCC: now also LED0.1 (VDD), LED1.1 (VDD), LED2.1 (VDD), LED3.1 (VDD), LED4.1 (VDD)
- new net: LED0.2 (DOUT), LED1.4 (DIN)
- new net: LED1.2 (DOUT), LED2.4 (DIN)
- new net: LED2.2 (DOUT), LED3.4 (DIN)
- new net: LED3.2 (DOUT), LED4.4 (DIN)
- no-connect marks 0 -> 9
Other:
- note added: "LEDS"
- moved on the sheet: JOLED0, SW0, SW1, U0

Commit message: create matrix
Parts:
- added D0, D1, D2, D3, D4, D5, D6, D7, D8, D9: DIODE, symbol Device:D_Small
- added SW10, SW2, SW3, SW4, SW5, SW6, SW7, SW8, SW9: SW_Push, symbol Switch:SW_Push
Connections:
- net C0: now also U0.16 (15/PB1); no longer U0.15 (14/PB3)
- net C1: now also U0.15 (14/PB3), SW2.2, SW5.2, SW8.2; no longer U0.14 (16/PB2)
- net C2: now also U0.14 (16/PB2), SW3.2, SW6.2, SW9.2; no longer U0.13 (10/PB6)
- net R0: now also D0.1 (K), D1.1 (K), D2.1 (K)
- net R1: now also D3.1 (K), D4.1 (K), D5.1 (K)
- net R2: now also D6.1 (K), D7.1 (K), D8.1 (K), D9.1 (K); no longer SW1.S1
- new net: D0.2 (A), SW2.1
- new net: D1.2 (A), SW3.1
- new net: D2.2 (A), SW4.1
- new net: D3.2 (A), SW5.1
- new net: D4.2 (A), SW6.1
- new net: D5.2 (A), SW7.1
- new net: D7.2 (A), SW8.1
- new net: D8.2 (A), SW9.1
- new net: D9.2 (A), SW10.1
- new net C3: SW10.2, SW4.2, SW7.2, U0.13 (10/PB6)
- new net ENR: D6.2 (A), SW1.S1
- no-connect marks 9 -> 8
Other:
- note added: "SWITCH MATRIX"
- moved on the sheet: LED0, LED1, LED2, LED3, LED4, U0

Commit message: update footprints fields
Parts:
- D0, D1, D2, D3, D4, D5, D6, D7, D8, D9: footprint (none) -> Keebio-Parts:MD_Diode
- JOLED0: footprint (none) -> Pin_Headers:Pin_Header_Straight_1x04_Pitch2.54mm
- LED0, LED1, LED2, LED3, LED4: footprint LED_SMD:LED_WS2812B_PLCC4_5.0x5.0mm_P3.2mm -> LEDs:LED_WS2812B-PLCC4
- SW0: footprint (none) -> Buttons_Switches_THT:SW_PUSH_6mm
- SW1: footprint (none) -> Keebio-Parts:RotaryEncoder_Alps_EC11E-Switch_Vertical_H20mm
- SW10, SW2, SW3, SW4, SW5, SW6, SW7, SW8, SW9: footprint (none) -> MX_Only:MXOnly-1U-Hotswap
- U0: footprint (none) -> Keebio-Parts:ArduinoProMicro

Commit message: pcb layout
Parts:
- added H0, H1, H2, H3: Hole, Mounting_Holes:MountingHole_2.2mm_M2, symbol keebio:Hole
Other:
- note added: "MOUNTING HOLES"
- moved on the sheet: U0
Changed lines of the file:
@@
 Wire Notes Line
 	6950 5600 6950 500
-NoConn ~ 5500 3100
-NoConn ~ 4100 3200
-NoConn ~ 4100 3100
-NoConn ~ 4100 3000
-NoConn ~ 4100 2500
-NoConn ~ 5500 2400
-NoConn ~ 5500 2800
-Wire Wire Line
-	4100 2400 4050 2400
-Text GLabel 5550 3400 2    50   Input ~ 0
-C2
-Text GLabel 5550 3300 2    50   Input ~ 0
-C1
-Text GLabel 5550 3200 2    50   Input ~ 0
-C0
-Wire Wire Line
-	4100 3500 4050 3500
-Wire Wire Line
-	4100 3400 4050 3400
-Text GLabel 4050 3500 0    50   Input ~ 0
-R2
-Text GLabel 4050 3400 0    50   Input ~ 0
-R1
-Wire Wire Line
-	4100 3300 4050 3300
-Text GLabel 4050 3300 0    50   Input ~ 0
-R0
-Wire Wire Line
-	5550 3000 5500 3000
-Wire Wire Line
-	5550 2900 5500 2900
-Text GLabel 5550 3000 2    50   Input ~ 0
-EN1
-Text GLabel 5550 2900 2    50   Input ~ 0
-EN0
-Text GLabel 4050 2400 0    50   Input ~ 0
-LEDS
-Wire Wire Line
-	4100 2900 4050 2900
-Text GLabel 4050 2900 0    50   Input ~ 0
-SCL
-Wire Wire Line
-	4100 2800 4050 2800
-Text GLabel 4050 2800 0    50   Input ~ 0
-SDA
-Connection ~ 4100 2600
-Wire Wire Line
-	4100 2600 4050 2600
-Wire Wire Line
-	5550 2500 5500 2500
-$Comp
-L power:GND #PWR0107
-U 1 1 5F039D77
-P 5550 2500
-F 0 "#PWR0107" H 5550 2250 50  0001 C CNN
-F 1 "GND" V 5555 2372 50  0000 R CNN
-F 2 "" H 5550 2500 50  0001 C CNN
-F 3 "" H 5550 2500 50  0001 C CNN
-	1    5550 2500
-	0    -1   -1   0
-$EndComp
-Wire Wire Line
-	5550 2700 5500 2700
-$Comp
-L power:VCC #PWR0108
-U 1 1 5F0416A0
-P 5550 2700
-F 0 "#PWR0108" H 5550 2550 50  0001 C CNN
-F 1 "VCC" V 5565 2828 50  0000 L CNN
-F 2 "" H 5550 2700 50  0001 C CNN
-F 3 "" H 5550 2700 50  0001 C CNN
-	1    5550 2700
-	0    1    1    0
-$EndComp
-Wire Wire Line
-	5550 2600 5500 2600
-Text GLabel 5550 2600 2    50   Input ~ 0
-RST
-Wire Wire Line
-	4100 2700 4100 2600
-$Comp
-L power:GND #PWR0109
-U 1 1 5F0376E2
-P 4050 2600
-F 0 "#PWR0109" H 4050 2350 50  0001 C CNN
-F 1 "GND" V 4055 2472 50  0000 R CNN
-F 2 "" H 4050 2600 50  0001 C CNN
-F 3 "" H 4050 2600 50  0001 C CNN
-	1    4050 2600
-	0    1    1    0
-$EndComp
-$Comp
-L keebio:ProMicro U0
-U 1 1 5F031D44
-P 4800 2950
-F 0 "U0" H 4800 3787 60  0000 C CNN
-F 1 "ProMicro" H 4800 3681 60  0000 C CNN
-F 2 "Keebio-Parts:ArduinoProMicro" V 5850 450 60  0001 C CNN
-F 3 "" V 5850 450 60  0001 C CNN
-	1    4800 2950
-	1    0    0    -1
-$EndComp
 Wire Wire Line
 	8650 3800 7850 3800
@@
 	1    0    0    -1
 $EndComp
-Text GLabel 5550 3500 2    50   Input ~ 0
-C3
 Text GLabel 8450 2400 1    50   Input ~ 0
 C0
@@
 	9050 3550 9050 4250
 Connection ~ 9050 3550
-Wire Wire Line
-	5550 3200 5500 3200
-Wire Wire Line
-	5550 3300 5500 3300
-Wire Wire Line
-	5550 3400 5500 3400
-Wire Wire Line
-	5500 3500 5550 3500
 $Comp
 L Device:Rotary_Encoder_Switch SW1
@@
 	1    0    0    -1
 $EndComp
+$Comp
+L keebio:Hole H0
+U 1 1 5F025C67
+P 3500 4750
+F 0 "H0" H 3686 4803 60  0000 L CNN
+F 1 "Hole" H 3686 4697 60  0000 L CNN
+F 2 "Mounting_Holes:MountingHole_2.2mm_M2" H 3500 4750 60  0001 C CNN
+F 3 "" H 3500 4750 60  0001 C CNN
+	1    3500 4750
+	1    0    0    -1
+$EndComp
+Text Notes 3050 4150 0    50   ~ 0
+MOUNTING HOLES
+Wire Notes Line
+	2850 3850 6900 3850
+NoConn ~ 5500 2250
+NoConn ~ 4100 2350
+NoConn ~ 4100 2250
+NoConn ~ 4100 2150
+NoConn ~ 4100 1650
+NoConn ~ 5500 1550
+NoConn ~ 5500 1950
+Wire Wire Line
+	4100 1550 4050 1550
+Text GLabel 5550 2550 2    50   Input ~ 0
+C2
+Text GLabel 5550 2450 2    50   Input ~ 0
+C1
+Text GLabel 5550 2350 2    50   Input ~ 0
+C0
+Wire Wire Line
+	4100 2650 4050 2650
+Wire Wire Line
+	4100 2550 4050 2550
+Text GLabel 4050 2650 0    50   Input ~ 0
+R2
+Text GLabel 4050 2550 0    50   Input ~ 0
+R1
+Wire Wire Line
+	4100 2450 4050 2450
+Text GLabel 4050 2450 0    50   Input ~ 0
+R0
+Wire Wire Line
+	5550 2150 5500 2150
+Wire Wire Line
+	5550 2050 5500 2050
+Text GLabel 5550 2150 2    50   Input ~ 0
+EN1
+Text GLabel 5550 2050 2    50   Input ~ 0
+EN0
+Text GLabel 4050 1550 0    50   Input ~ 0
+LEDS
+Wire Wire Line
+	4100 2050 4050 2050
+Text GLabel 4050 2050 0    50   Input ~ 0
+SCL
+Wire Wire Line
+	4100 1950 4050 1950
+Text GLabel 4050 1950 0    50   Input ~ 0
+SDA
+Connection ~ 4100 1750
+Wire Wire Line
+	4100 1750 4050 1750
+Wire Wire Line
+	5550 1650 5500 1650
+$Comp
+L power:GND #PWR0107
+U 1 1 5F039D77
+P 5550 1650
+F 0 "#PWR0107" H 5550 1400 50  0001 C CNN
+F 1 "GND" V 5555 1522 50  0000 R CNN
+F 2 "" H 5550 1650 50  0001 C CNN
+F 3 "" H 5550 1650 50  0001 C CNN
+	1    5550 1650
+	0    -1   -1   0
+$EndComp
+Wire Wire Line
+	5550 1850 5500 1850
+$Comp
+L power:VCC #PWR0108
+U 1 1 5F0416A0
+P 5550 1850
+F 0 "#PWR0108" H 5550 1700 50  0001 C CNN
+F 1 "VCC" V 5565 1978 50  0000 L CNN
+F 2 "" H 5550 1850 50  0001 C CNN
+F 3 "" H 5550 1850 50  0001 C CNN
+	1    5550 1850
+	0    1    1    0
+$EndComp
+Wire Wire Line
+	5550 1750 5500 1750
+Text GLabel 5550 1750 2    50   Input ~ 0
+RST
+Wire Wire Line
+	4100 1850 4100 1750
+$Comp
+L power:GND #PWR0109
+U 1 1 5F0376E2
+P 4050 1750
+F 0 "#PWR0109" H 4050 1500 50  0001 C CNN
+F 1 "GND" V 4055 1622 50  0000 R CNN
+F 2 "" H 4050 1750 50  0001 C CNN
+F 3 "" H 4050 1750 50  0001 C CNN
+	1    4050 1750
+	0    1    1    0
+$EndComp
+$Comp
+L keebio:ProMicro U0
+U 1 1 5F031D44
+P 4800 2100
+F 0 "U0" H 4800 2937 60  0000 C CNN
+F 1 "ProMicro" H 4800 2831 60  0000 C CNN
+F 2 "Keebio-Parts:ArduinoProMicro" V 5850 -400 60  0001 C CNN
+F 3 "" V 5850 -400 60  0001 C CNN
+	1    4800 2100
+	1    0    0    -1
+$EndComp
+Text GLabel 5550 2650 2    50   Input ~ 0
+C3
+Wire Wire Line
+	5550 2350 5500 2350
+Wire Wire Line
+	5550 2450 5500 2450
+Wire Wire Line
+	5550 2550 5500 2550
+Wire Wire Line
+	5500 2650 5550 2650
+$Comp
+L keebio:Hole H1
+U 1 1 5F03A4BC
+P 4350 4750
+F 0 "H1" H 4536 4803 60  0000 L CNN
+F 1 "Hole" H 4536 4697 60  0000 L CNN
+F 2 "Mounting_Holes:MountingHole_2.2mm_M2" H 4350 4750 60  0001 C CNN
+F 3 "" H 4350 4750 60  0001 C CNN
+	1    4350 4750
+	1    0    0    -1
+$EndComp
+$Comp
+L keebio:Hole H2
+U 1 1 5F03ADC0
+P 5200 4750
+F 0 "H2" H 5386 4803 60  0000 L CNN
+F 1 "Hole" H 5386 4697 60  0000 L CNN
+F 2 "Mounting_Holes:MountingHole_2.2mm_M2" H 5200 4750 60  0001 C CNN
+F 3 "" H 5200 4750 60  0001 C CNN
+	1    5200 4750
+	1    0    0    -1
+$EndComp
+$Comp
+L keebio:Hole H3
+U 1 1 5F03BD3F
+P 6050 4750
+F 0 "H3" H 6236 4803 60  0000 L CNN
+F 1 "Hole" H 6236 4697 60  0000 L CNN
+F 2 "Mounting_Holes:MountingHole_2.2mm_M2" H 6050 4750 60  0001 C CNN
+F 3 "" H 6050 4750 60  0001 C CNN
+	1    6050 4750
+	1    0    0    -1
+$EndComp
